File: pcb/iso.sch (KiCad schematic (older format))
At the start: 19 parts, among them J1 Conn_01x06, U1 ATmega328P-AU, U2 SRV05-4, X1 Crystal_GND24_Small

Commit message: RGB!!!
Parts:
- removed MX1: MX-LED, MX_Only:MXOnly-ISO-ReversedStabilizers, symbol MX_Alps_Hybrid:MX-LED
- removed R7: 1k, Resistor_SMD:R_0805_2012Metric, symbol Device:R_Small
- added LED1, LED2, LED3: SK6812MINI, custom_parts:SK6812MINIE-simple, symbol LED:SK6812MINI
- added MX1: MX-NoLED, custom_parts:MXOnly-ISO-ROTATEDCCW-ReversedStabilizers-NoLED, symbol MX_Alps_Hybrid:MX-NoLED
- C1: footprint Capacitor_SMD:C_0805_2012Metric -> Capacitor_SMD:C_0603_1608Metric; LCSC C91245 -> C57112
- C7, C8: footprint Capacitor_SMD:C_0805_2012Metric -> Capacitor_SMD:C_0603_1608Metric; LCSC C1804 -> C1653
- D1, D2: footprint Diode_SMD:D_SOD-123 -> Diode_SMD:D_SOD-323; LCSC C173412 -> C401091
- R1, R2: footprint Resistor_SMD:R_0805_2012Metric -> Resistor_SMD:R_0603_1608Metric; LCSC C27834 -> C23186
- R3: footprint Resistor_SMD:R_0805_2012Metric -> Resistor_SMD:R_0603_1608Metric; LCSC C4310 -> C22843
- R4, R5: footprint Resistor_SMD:R_0805_2012Metric -> Resistor_SMD:R_0603_1608Metric; LCSC C17802 -> C27592
Connections:
- net +5V: now also LED1.4 (VDD), LED2.4 (VDD), LED3.4 (VDD)
- net GND: now also LED1.2 (VSS), LED2.2 (VSS), LED3.2 (VSS), MX1.2 (ROW)
- net LED: now also U1.14 (PB2), LED1.3 (DIN); no longer U1.13 (PB1)
- net SW: now also U1.12 (PB0), MX1.1 (COL); no longer U1.10 (PD6)
- net at D1.1 (K), R3.1, R4.2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: now also U2.4 (IO3); no longer U2.3 (IO2)
- net at D2.1 (K), R5.2, USB1.A6 (D+)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: now also U2.1 (IO1); no longer U2.6 (IO4)
- new net: LED1.1 (DOUT), LED2.3 (DIN)
- new net: LED2.1 (DOUT), LED3.3 (DIN)
Changed lines of the file:
@@
 F 0 "C1" H 1392 9846 50  0000 L CNN
 F 1 "10uF" H 1392 9755 50  0000 L CNN
-F 2 "Capacitor_SMD:C_0805_2012Metric" H 1300 9800 50  0001 C CNN
+F 2 "Capacitor_SMD:C_0603_1608Metric" H 1300 9800 50  0001 C CNN
 F 3 "~" H 1300 9800 50  0001 C CNN
-F 4 "C91245" H 1300 9800 50  0001 C CNN "LCSC"
+F 4 "C57112" H 1300 9800 50  0001 C CNN "LCSC"
 	1    1300 9800
 	1    0    0    -1
@@
 F 0 "C7" V 3571 3300 50  0000 C CNN
 F 1 "22pF" V 3662 3300 50  0000 C CNN
-F 2 "Capacitor_SMD:C_0805_2012Metric" H 3800 3300 50  0001 C CNN
+F 2 "Capacitor_SMD:C_0603_1608Metric" H 3800 3300 50  0001 C CNN
 F 3 "~" H 3800 3300 50  0001 C CNN
-F 4 "C1804" V 3800 3300 50  0001 C CNN "LCSC"
+F 4 "C1653" V 3800 3300 50  0001 C CNN "LCSC"
 	1    3800 3300
 	0    -1   -1   0
@@
 F 0 "C8" V 3571 2950 50  0000 C CNN
 F 1 "22pF" V 3662 2950 50  0000 C CNN
-F 2 "Capacitor_SMD:C_0805_2012Metric" H 3800 2950 50  0001 C CNN
+F 2 "Capacitor_SMD:C_0603_1608Metric" H 3800 2950 50  0001 C CNN
 F 3 "~" H 3800 2950 50  0001 C CNN
-F 4 "C1804" V 3800 2950 50  0001 C CNN "LCSC"
+F 4 "C1653" V 3800 2950 50  0001 C CNN "LCSC"
 	1    3800 2950
 	0    -1   -1   0
@@
 F 0 "R1" V 3800 9150 50  0000 C CNN
 F 1 "5.1k" V 3700 9150 50  0000 C CNN
-F 2 "Resistor_SMD:R_0805_2012Metric" H 3800 9150 50  0001 C CNN
+F 2 "Resistor_SMD:R_0603_1608Metric" H 3800 9150 50  0001 C CNN
 F 3 "~" H 3800 9150 50  0001 C CNN
-F 4 "C27834" V 3800 9150 50  0001 C CNN "LCSC"
+F 4 "C23186" V 3800 9150 50  0001 C CNN "LCSC"
 	1    3800 9150
 	0    1    1    0
@@
 F 0 "R2" V 4000 9250 50  0000 C CNN
 F 1 "5.1k" V 3895 9250 50  0000 C CNN
-F 2 "Resistor_SMD:R_0805_2012Metric" H 4000 9250 50  0001 C CNN
+F 2 "Resistor_SMD:R_0603_1608Metric" H 4000 9250 50  0001 C CNN
 F 3 "~" H 4000 9250 50  0001 C CNN
-F 4 "C27834" V 4000 9250 50  0001 C CNN "LCSC"
+F 4 "C23186" V 4000 9250 50  0001 C CNN "LCSC"
 	1    4000 9250
 	0    1    1    0
@@
 F 0 "R4" V 5100 9450 50  0000 C CNN
 F 1 "68R" V 4995 9450 50  0000 C CNN
-F 2 "Resistor_SMD:R_0805_2012Metric" H 5100 9450 50  0001 C CNN
+F 2 "Resistor_SMD:R_0603_1608Metric" H 5100 9450 50  0001 C CNN
 F 3 "~" H 5100 9450 50  0001 C CNN
-F 4 "C17802" V 5100 9450 50  0001 C CNN "LCSC"
+F 4 "C27592" V 5100 9450 50  0001 C CNN "LCSC"
 	1    5100 9450
 	0    1    1    0
@@
 F 0 "R5" V 5100 9650 50  0000 C CNN
 F 1 "68R" V 5000 9650 50  0000 C CNN
-F 2 "Resistor_SMD:R_0805_2012Metric" H 5100 9650 50  0001 C CNN
+F 2 "Resistor_SMD:R_0603_1608Metric" H 5100 9650 50  0001 C CNN
 F 3 "~" H 5100 9650 50  0001 C CNN
-F 4 "C17802" V 5100 9650 50  0001 C CNN "LCSC"
+F 4 "C27592" V 5100 9650 50  0001 C CNN "LCSC"
 	1    5100 9650
 	0    1    1    0
@@
 F 0 "D2" V 4404 10120 50  0000 L CNN
 F 1 "D_Zener_Small" V 4495 10120 50  0000 L CNN
-F 2 "Diode_SMD:D_SOD-123" V 4450 10050 50  0001 C CNN
+F 2 "Diode_SMD:D_SOD-323" V 4450 10050 50  0001 C CNN
 F 3 "~" V 4450 10050 50  0001 C CNN
-F 4 "C173412" H 4450 10050 50  0001 C CNN "LCSC"
+F 4 "C401091" H 4450 10050 50  0001 C CNN "LCSC"
 	1    4450 10050
 	0    1    1    0
@@
 F 0 "D1" V 4154 10120 50  0000 L CNN
 F 1 "D_Zener_Small" V 4245 10120 50  0000 L CNN
-F 2 "Diode_SMD:D_SOD-123" V 4200 10050 50  0001 C CNN
+F 2 "Diode_SMD:D_SOD-323" V 4200 10050 50  0001 C CNN
 F 3 "~" V 4200 10050 50  0001 C CNN
-F 4 "C173412" H 4200 10050 50  0001 C CNN "LCSC"
+F 4 "C401091" H 4200 10050 50  0001 C CNN "LCSC"
 	1    4200 10050
 	0    1    1    0
@@
 F 0 "R3" V 4600 9200 50  0000 C CNN
 F 1 "1.5K" V 4495 9200 50  0000 C CNN
-F 2 "Resistor_SMD:R_0805_2012Metric" H 4600 9200 50  0001 C CNN
+F 2 "Resistor_SMD:R_0603_1608Metric" H 4600 9200 50  0001 C CNN
 F 3 "~" H 4600 9200 50  0001 C CNN
-F 4 "C4310" V 4600 9200 50  0001 C CNN "LCSC"
+F 4 "C22843" V 4600 9200 50  0001 C CNN "LCSC"
 	1    4600 9200
 	-1   0    0    1
@@
 Wire Wire Line
 	1300 9700 1300 9550
-$Comp
-L MX_Alps_Hybrid:MX-LED MX1
-U 1 1 615021F8
-P 4900 2350
-F 0 "MX1" H 4982 2574 60  0000 C CNN
-F 1 "MX-LED" H 4982 2500 20  0000 C CNN
-F 2 "MX_Only:MXOnly-ISO-ReversedStabilizers" H 4275 2325 60  0001 C CNN
-F 3 "" H 4275 2325 60  0001 C CNN
-	1    4900 2350
-	1    0    0    -1
-$EndComp
 Text GLabel 5250 2250 2    50   Input ~ 0
 SW
@@
 Wire Wire Line
 	5150 2250 5250 2250
-Text GLabel 5250 2400 2    50   Input ~ 0
-LED
-Wire Wire Line
-	5250 2400 5150 2400
-Wire Wire Line
-	5150 2400 5150 2350
-Wire Wire Line
-	5150 2350 5000 2350
-$Comp
-L power:GND #PWR0104
-U 1 1 61505E3F
-P 5000 2800
-F 0 "#PWR0104" H 5000 2550 50  0001 C CNN
-F 1 "GND" H 5005 2627 50  0000 C CNN
-F 2 "" H 5000 2800 50  0001 C CNN
-F 3 "" H 5000 2800 50  0001 C CNN
-	1    5000 2800
-	1    0    0    -1
-$EndComp
-$Comp
-L Device:R_Small R7
-U 1 1 61506847
-P 5000 2600
-F 0 "R7" H 4941 2554 50  0000 R CNN
-F 1 "1k" H 4941 2645 50  0000 R CNN
-F 2 "Resistor_SMD:R_0805_2012Metric" H 5000 2600 50  0001 C CNN
-F 3 "~" H 5000 2600 50  0001 C CNN
-F 4 "C17513" H 5000 2600 50  0001 C CNN "LCSC"
-	1    5000 2600
-	-1   0    0    1
-$EndComp
-Wire Wire Line
-	5000 2800 5000 2700
-Wire Wire Line
-	5000 2500 5000 2450
-Wire Wire Line
-	5000 2450 4900 2450
 Wire Wire Line
 	5800 9550 5950 9550
@@
 L power:GND #PWR0101
 U 1 1 6134E819
-P 5800 9550
-F 0 "#PWR0101" H 5800 9300 50  0001 C CNN
-F 1 "GND" H 5805 9377 50  0000 C CNN
-F 2 "" H 5800 9550 50  0001 C CNN
-F 3 "" H 5800 9550 50  0001 C CNN
-	1    5800 9550
+P 7100 9550
+F 0 "#PWR0101" H 7100 9300 50  0001 C CNN
+F 1 "GND" H 7105 9377 50  0000 C CNN
+F 2 "" H 7100 9550 50  0001 C CNN
+F 3 "" H 7100 9550 50  0001 C CNN
+	1    7100 9550
 	1    0    0    -1
 $EndComp
@@
 F 4 "C85364" H 6450 9550 50  0001 C CNN "LCSC"
 	1    6450 9550
-	0    1    1    0
+	0    -1   -1   0
 $EndComp
 $Comp
 L power:VCC #PWR0102
 U 1 1 61520AA9
-P 7100 9550
-F 0 "#PWR0102" H 7100 9400 50  0001 C CNN
-F 1 "VCC" H 7115 9723 50  0000 C CNN
-F 2 "" H 7100 9550 50  0001 C CNN
-F 3 "" H 7100 9550 50  0001 C CNN
-	1    7100 9550
-	1    0    0    -1
-$EndComp
-Text GLabel 2450 4550 2    50   Input ~ 0
+P 5800 9550
+F 0 "#PWR0102" H 5800 9400 50  0001 C CNN
+F 1 "VCC" H 5815 9723 50  0000 C CNN
+F 2 "" H 5800 9550 50  0001 C CNN
+F 3 "" H 5800 9550 50  0001 C CNN
+	1    5800 9550
+	1    0    0    -1
+$EndComp
+Text GLabel 2450 2250 2    50   Input ~ 0
 SW
-Text GLabel 2450 2350 2    50   Input ~ 0
+Text GLabel 2450 2450 2    50   Input ~ 0
 LED
 $Comp
-L power:GND #PWR?
+L power:GND #PWR0105
 U 1 1 61580668
 P 4650 2550
-F 0 "#PWR?" H 4650 2300 50  0001 C CNN
+F 0 "#PWR0105" H 4650 2300 50  0001 C CNN
 F 1 "GND" H 4655 2377 50  0000 C CNN
 F 2 "" H 4650 2550 50  0001 C CNN
@@
 Wire Wire Line
 	4650 2500 4650 2550
+$Comp
+L LED:SK6812MINI LED1
+U 1 1 614BBA26
+P 5150 4450
+F 0 "LED1" H 5300 4850 50  0000 L CNN
+F 1 "SK6812MINI" H 5300 4750 50  0000 L CNN
+F 2 "custom_parts:SK6812MINIE-simple" H 5200 4150 50  0001 L TNN
+F 3 "https://cdn-shop.adafruit.com/product-files/2686/SK6812MINI_REV.01-1-2.pdf" H 5250 4075 50  0001 L TNN
+	1    5150 4450
+	1    0    0    -1
+$EndComp
+$Comp
+L power:GND #PWR0111
+U 1 1 614BC3E0
+P 5150 4750
+F 0 "#PWR0111" H 5150 4500 50  0001 C CNN
+F 1 "GND" H 5155 4577 50  0000 C CNN
+F 2 "" H 5150 4750 50  0001 C CNN
+F 3 "" H 5150 4750 50  0001 C CNN
+	1    5150 4750
+	1    0    0    -1
+$EndComp
+$Comp
+L power:+5V #PWR0112
+U 1 1 614BCE02
+P 5150 4150
+F 0 "#PWR0112" H 5150 4000 50  0001 C CNN
+F 1 "+5V" H 5165 4323 50  0000 C CNN
+F 2 "" H 5150 4150 50  0001 C CNN
+F 3 "" H 5150 4150 50  0001 C CNN
+	1    5150 4150
+	1    0    0    -1
+$EndComp
+Text GLabel 4850 4450 0    50   Input ~ 0
+LED
+$Comp
+L MX_Alps_Hybrid:MX-NoLED MX1
+U 1 1 614BF2DA
+P 4900 2350
+F 0 "MX1" H 4933 2573 60  0000 C CNN
+F 1 "MX-NoLED" H 4933 2499 20  0000 C CNN
+F 2 "custom_parts:MXOnly-ISO-ROTATEDCCW-ReversedStabilizers-NoLED" H 4275 2325 60  0001 C CNN
+F 3 "" H 4275 2325 60  0001 C CNN
+	1    4900 2350
+	1    0    0    -1
+$EndComp
+Connection ~ 7100 9550
+$Comp
+L LED:SK6812MINI LED2
+U 1 1 61500DC0
+P 5750 4450
+F 0 "LED2" H 5900 4850 50  0000 L CNN
+F 1 "SK6812MINI" H 5900 4750 50  0000 L CNN
+F 2 "custom_parts:SK6812MINIE-simple" H 5800 4150 50  0001 L TNN
+F 3 "https://cdn-shop.adafruit.com/product-files/2686/SK6812MINI_REV.01-1-2.pdf" H 5850 4075 50  0001 L TNN
+	1    5750 4450
+	1    0    0    -1
+$EndComp
+$Comp
+L LED:SK6812MINI LED3
+U 1 1 61501412
+P 6350 4450
+F 0 "LED3" H 6500 4850 50  0000 L CNN
+F 1 "SK6812MINI" H 6500 4750 50  0000 L CNN
+F 2 "custom_parts:SK6812MINIE-simple" H 6400 4150 50  0001 L TNN
+F 3 "https://cdn-shop.adafruit.com/product-files/2686/SK6812MINI_REV.01-1-2.pdf" H 6450 4075 50  0001 L TNN
+	1    6350 4450
+	1    0    0    -1
+$EndComp
+$Comp
+L power:+5V #PWR0104
+U 1 1 61501BB8
+P 5750 4150
+F 0 "#PWR0104" H 5750 4000 50  0001 C CNN
+F 1 "+5V" H 5765 4323 50  0000 C CNN
+F 2 "" H 5750 4150 50  0001 C CNN
+F 3 "" H 5750 4150 50  0001 C CNN
+	1    5750 4150
+	1    0    0    -1
+$EndComp
+$Comp
+L power:+5V #PWR0113
+U 1 1 6150201A
+P 6350 4150
+F 0 "#PWR0113" H 6350 4000 50  0001 C CNN
+F 1 "+5V" H 6365 4323 50  0000 C CNN
+F 2 "" H 6350 4150 50  0001 C CNN
+F 3 "" H 6350 4150 50  0001 C CNN
+	1    6350 4150
+	1    0    0    -1
+$EndComp
+$Comp
+L power:GND #PWR0114
+U 1 1 61502564
+P 5750 4750
+F 0 "#PWR0114" H 5750 4500 50  0001 C CNN
+F 1 "GND" H 5755 4577 50  0000 C CNN
+F 2 "" H 5750 4750 50  0001 C CNN
+F 3 "" H 5750 4750 50  0001 C CNN
+	1    5750 4750
+	1    0    0    -1
+$EndComp
+$Comp
+L power:GND #PWR0115
+U 1 1 61502A8C
+P 6350 4750
+F 0 "#PWR0115" H 6350 4500 50  0001 C CNN
+F 1 "GND" H 6355 4577 50  0000 C CNN
+F 2 "" H 6350 4750 50  0001 C CNN
+F 3 "" H 6350 4750 50  0001 C CNN
+	1    6350 4750
+	1    0    0    -1
+$EndComp
 $EndSCHEMATC

Commit message: update
Parts:
- C1: LCSC C57112 -> C19702
Changed lines of the file:
@@
 F 2 "Capacitor_SMD:C_0603_1608Metric" H 1300 9800 50  0001 C CNN
 F 3 "~" H 1300 9800 50  0001 C CNN
-F 4 "C57112" H 1300 9800 50  0001 C CNN "LCSC"
+F 4 "C19702" H 1300 9800 50  0001 C CNN "LCSC"
 	1    1300 9800
 	1    0    0    -1
